File: phoenix-adapter/phoenix-adapter.sch (KiCad schematic (older format))
At the start: 0 parts

Commit message: prelim pcb done, waiting on feedback from the boyz!
Parts:
- added CON101: RCJ-2223, db-thparts:RCJ-2223, symbol RCJ-2223
Connections:
- net labels added: GND, LEFT, RIGHT
- wire segments 0 -> 3
Changed lines of the file:
@@
 LIBS:db-transistors
 LIBS:db-vgparts
+LIBS:phoenix-adapter-cache
 EELAYER 25 0
 EELAYER END
@@
 EndData
 $EndBitmap
+$Comp
+L RCJ-2223 CON101
+U 1 1 5ABE576C
+P 5250 2950
+F 0 "CON101" H 5350 3025 50  0000 C CNN
+F 1 "RCJ-2223" H 5450 3100 50  0000 C CNN
+F 2 "db-thparts:RCJ-2223" H 5775 3525 60  0001 C CNN
+F 3 "https://www.cui.com/product/resource/rcj-22xx.pdf" H 6475 3225 60  0001 C CNN
+F 4 "CP-1435-ND" H 5575 3325 60  0001 C CNN "Digikey"
+F 5 "CONN RCA JACK MONO 3.2MM R/A" H 6050 3425 60  0001 C CNN "Description"
+	1    5250 2950
+	1    0    0    -1
+$EndComp
+$Comp
+L GND #PWR?
+U 1 1 5ABE5F05
+P 5250 3450
+F 0 "#PWR?" H 5250 3200 50  0001 C CNN
+F 1 "GND" H 5250 3300 50  0000 C CNN
+F 2 "" H 5250 3450 50  0001 C CNN
+F 3 "" H 5250 3450 50  0001 C CNN
+	1    5250 3450
+	1    0    0    -1
+$EndComp
+Wire Wire Line
+	5600 3175 5950 3175
+Wire Wire Line
+	5600 3025 5950 3025
+Wire Wire Line
+	5250 3325 5250 3450
+Text Label 5650 3175 0    60   ~ 0
+LEFT
+Text Label 5650 3025 0    60   ~ 0
+RIGHT
 $EndSCHEMATC
